File: HAMKey-One.kicad_sch (KiCad schematic)
At the start: 59 parts, among them J1 Conn_01x04, Q1 DTC143Z, SW1 SW_Main, SW2 SW_Reset, SW3 SW_PWR, U1 nRF52832-QFxx, Y1 Xtal_32M, Y2 32.768kHz

Commit message: near finish layout
Parts:
- removed AE1: Antenna, symbol Device:Antenna
- removed U2: ~, Package_DFN_QFN:DFN-8-1EP_3x3mm_P0.65mm_EP1.55x2.4mm, symbol nigh_Library:LP4073
- added AE1: Antenna_Shield, RF_Antenna:Texas_SWRA117D_2.4GHz_Right, symbol Device:Antenna_Shield
- added C20, C21: 0.47uF, Capacitor_SMD:C_0402_1005Metric_Pad0.74x0.62mm_HandSolder, symbol Device:C_Small
- added SW4, SW5: SW_Main, xianii:KEY-1511, symbol Switch:SW_Push
- added SW6: SW_SOUND, xianii:SK-3296S-01-L1, symbol Switch:SW_SPDT
- added U2: SLM6400, Package_DFN_QFN:DFN-8-1EP_3x3mm_P0.65mm_EP1.55x2.4mm, symbol nigh_Library:SLM6400
- BATT1: footprint nigh_Library:BATT2030 -> xianii:BATT-501240
- BZ1: footprint nigh_Library:buzzer_SMD -> xianii:BUZZ-9032
- C1, C2, C3, C4: footprint Capacitor_SMD:C_0402_1005Metric_Pad0.74x0.62mm_HandSolder -> Capacitor_SMD:C_0402_1005Metric
- C10, C11, C12, C13, C14, C15, C16, C17, C18, C19, C5, C6, C7, C8, C9: footprint Capacitor_SMD:C_0603_1608Metric_Pad1.08x0.95mm_HandSolder -> Capacitor_SMD:C_0402_1005Metric
- J1: footprint Connector_PinHeader_2.54mm:PinHeader_1x04_P2.54mm_Horizontal -> Connector_PinHeader_2.54mm:PinHeader_1x04_P2.54mm_Vertical
- L1: footprint (none) -> Inductor_SMD:L_0603_1608Metric
- L2: footprint (none) -> Inductor_SMD:L_0402_1005Metric
- R1, R10, R11, R12, R13, R14, R15, R16, R17, R2, R3, R4, R5, R6, R7, R9: footprint Resistor_SMD:R_0402_1005Metric_Pad0.72x0.64mm_HandSolder -> Resistor_SMD:R_0402_1005Metric
- SW1: footprint Button_Switch_Keyboard:SW_Cherry_MX_1.00u_PCB -> xianii:KEY-1511
- SW2: footprint (none) -> Jumper:SolderJumper-2_P1.3mm_Open_TrianglePad1.0x1.5mm
- U3: footprint Package_TO_SOT_SMD:TSOT-23_HandSoldering -> Package_TO_SOT_SMD:SOT-23
- Y1: footprint (none) -> PCM_Crystal_AKL:Crystal_SMD_2016-4Pin_2.0x1.6mm
- Y2: footprint (none) -> PCM_Crystal_AKL:Crystal_SMD_3215-2Pin_3.2x1.5mm
Connections:
- net ON/OFF is gone; now on net +3.3V: SW3.2 (B)
- net +3.3V: now also SW4.2, SW5.2; no longer C7.1, SW3.1 (A), U3.2 (VOUT)
- net +5V: now also C8.2, U2.4 (VCC); no longer C8.1
- net BAT+: now also U2.5 (BAT)
- net BUZZER: now also U1.17 (P0.14); no longer U1.9 (P0.07)
- net CHARGING: now also D6.1 (K), U2.7 (~{CHRG})
- net GND: now also C8.1, R10.1, AE1.2 (Shield), C20.1, C21.1, SW6.3 (C), U2.3 (GND), U2.8 (~{CE}), U2.9 (EP); no longer C8.2, R10.2
- net SWDP: now reaches J1.2 (Pin_2), R6.2
- net at C17.1, R17.1: now also AE1.1 (A)
- net SWDN: now reaches J1.3 (Pin_3), R7.2
- net SW_SOUND: now reaches U1.10 (P0.08)
- net SW_SOUND: now also SW6.2 (B)
- net BTN2: now reaches U1.19 (P0.16)
- net BTN2: now also C21.2, SW5.1
- net BTN0: now reaches U1.20 (P0.17)
- net BTN0: now also C3.2, SW1.1, C20.2, SW4.1
- removed net BTN: C3.2, SW1.1, U1.8 (P0.06)
- removed net LED_GREEN: D6.1 (K), U1.17 (P0.14)
- net SWDCLK renamed SWD+
- net SWDIO renamed SWD-
- new net: R10.2, U2.2 (PROG)
- new net LDO3v3: C7.1, SW3.1 (A), SW6.1 (A), U3.2 (VOUT)
Other:
- moved on the sheet: BATT1, BZ1, C3, C4, C6, C8, D3, D4, D5, D6, J1, Q1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

Commit message: first production ver
Parts:
- added FID1, FID2: Fiducial, xianii:marker1, symbol Mechanical:Fiducial
- D3, D4, D5, D6: footprint LED_SMD:LED_0402_1005Metric_Pad0.77x0.64mm_HandSolder -> LED_SMD:LED_0402_1005Metric
- R13, R16: value 470R -> 390R
- R14: value 470R -> 47R
- R15: value 470R -> 75R
- SW3: footprint nigh_Library:SS12D06G5 -> xianii:SS12D06G5
- U3: value ~ -> ME6210A33M3G
- USB1: footprint nigh_Library:Type-C-3.2H -> xianii:Type-C-3.2H
Changed lines of the file:
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@@
 			)
 		)
-		(property "Footprint" "LED_SMD:LED_0402_1005Metric_Pad0.77x0.64mm_HandSolder"
+		(property "Footprint" "LED_SMD:LED_0402_1005Metric"
 			(at 250.19 143.51 0)
 			(effects
@@
 			)
 		)
-		(property "Footprint" "LED_SMD:LED_0402_1005Metric_Pad0.77x0.64mm_HandSolder"
+		(property "Footprint" "LED_SMD:LED_0402_1005Metric"
 			(at 250.19 158.75 0)
 			(effects
@@
 	)
 	(symbol
+		(lib_id "Mechanical:Fiducial")
+		(at 273.05 54.61 0)
+		(unit 1)
+		(exclude_from_sim yes)
+		(in_bom no)
+		(on_board yes)
+		(dnp no)
+		(fields_autoplaced yes)
+		(property "Reference" "FID2"
+			(at 275.59 53.3399 0)
+			(effects
+				(font
+					(size 1.27 1.27)
+				)
+				(justify left)
+			)
+		)
+		(property "Value" "Fiducial"
+			(at 275.59 55.8799 0)
+			(effects
+				(font
+					(size 1.27 1.27)
+				)
+				(justify left)
+			)
+		)
+		(property "Footprint" "xianii:marker1"
+			(at 273.05 54.61 0)
+			(effects
+				(font
+					(size 1.27 1.27)
+				)
+				(hide yes)
+			)
+		)
+		(property "Datasheet" "~"
+			(at 273.05 54.61 0)
+			(effects
+				(font
+					(size 1.27 1.27)
+				)
+				(hide yes)
+			)
+		)
+		(property "Description" "Fiducial Marker"
+			(at 273.05 54.61 0)
+			(effects
+				(font
+					(size 1.27 1.27)
+				)
+				(hide yes)
+			)
+		)
+		(instances
+			(project "HAMKey-One"
+				(path "/613fe7f2-55f8-4770-afca-1b2f2a94adcb"
+					(reference "FID2")
+					(unit 1)
+				)
+			)
+		)
+	)
+	(symbol
 		(lib_id "power:GND")
 		(at 208.28 121.92 90)
@@
 			)
 		)
-		(property "Footprint" "LED_SMD:LED_0402_1005Metric_Pad0.77x0.64mm_HandSolder"
+		(property "Footprint" "LED_SMD:LED_0402_1005Metric"
 			(at 250.19 153.67 0)
 			(effects
@@
 			)
 		)
-		(property "Value" "470R"
+		(property "Value" "390R"
 			(at 267.462 144.78 90)
 			(effects
@@
 	)
 	(symbol
+		(lib_id "Mechanical:Fiducial")
+		(at 273.05 49.53 0)
+		(unit 1)
+		(exclude_from_sim yes)
+		(in_bom no)
+		(on_board yes)
+		(dnp no)
+		(fields_autoplaced yes)
+		(property "Reference" "FID1"
+			(at 275.59 48.2599 0)
+			(effects
+				(font
+					(size 1.27 1.27)
+				)
+				(justify left)
+			)
+		)
+		(property "Value" "Fiducial"
+			(at 275.59 50.7999 0)
+			(effects
+				(font
+					(size 1.27 1.27)
+				)
+				(justify left)
+			)
+		)
+		(property "Footprint" "xianii:marker1"
+			(at 273.05 49.53 0)
+			(effects
+				(font
+					(size 1.27 1.27)
+				)
+				(hide yes)
+			)
+		)
+		(property "Datasheet" "~"
+			(at 273.05 49.53 0)
+			(effects
+				(font
+					(size 1.27 1.27)
+				)
+				(hide yes)
+			)
+		)
+		(property "Description" "Fiducial Marker"
+			(at 273.05 49.53 0)
+			(effects
+				(font
+					(size 1.27 1.27)
+				)
+				(hide yes)
+			)
+		)
+		(instances
+			(project ""
+				(path "/613fe7f2-55f8-4770-afca-1b2f2a94adcb"
+					(reference "FID1")
+					(unit 1)
+				)
+			)
+		)
+	)
+	(symbol
 		(lib_id "Switch:SW_SPDT")
 		(at 200.66 97.79 0)
@@
 			)
 		)
-		(property "Footprint" "nigh_Library:SS12D06G5"
+		(property "Footprint" "xianii:SS12D06G5"
 			(at 200.66 97.79 0)
 			(effects
@@
 			)
 		)
-		(property "Value" "470R"
+		(property "Value" "47R"
 			(at 267.462 149.86 90)
 			(effects
@@
 			)
 		)
-		(property "Value" "~"
-			(at 243.84 21.59 0)
+		(property "Value" "ME6210A33M3G"
+			(at 239.268 20.32 0)
 			(effects
 				(font
@@
 			)
 		)
-		(property "Value" "470R"
+		(property "Value" "390R"
 			(at 267.462 160.02 90)
 			(effects
@@
 			)
 		)
-		(property "Footprint" "nigh_Library:Type-C-3.2H"
+		(property "Footprint" "xianii:Type-C-3.2H"
 			(at 69.85 165.1 0)
 			(effects
@@
 			)
 		)
-		(property "Value" "470R"
+		(property "Value" "75R"
 			(at 267.462 154.94 90)
 			(effects
@@
 			)
 		)
-		(property "Footprint" "LED_SMD:LED_0402_1005Metric_Pad0.77x0.64mm_HandSolder"
+		(property "Footprint" "LED_SMD:LED_0402_1005Metric"
 			(at 250.19 148.59 0)
 			(effects
